File: PCB/KiCad/Splitflap/Splitflap.kicad_pcb (KiCad board)
At the start: 2 copper layers, 40 x 80 mm, 18 parts, among them J1 Conn_01x05, J2 Conn_01x03, J3_In1 Conn_01x04, J4_Out1 Conn_01x04, Q1 BSS138, Q2 BSS138, U1 ESP8266-01_ESP-01, U2 L7805, U3 ULN2003A, U4 AMS1117-3.3

Commit message: 5v variante
Parts:
- removed C2, C3: C, Capacitor_THT:CP_Radial_D4.0mm_P2.00mm
- removed U2: L7805, Package_TO_SOT_THT:TO-220-3_Vertical
- U3: footprint Package_SO:SOP-16_4.55x10.3mm_P1.27mm -> Package_DIP:DIP-16_W7.62mm; moved to F.Cu
- moved U3 13.5 mm to (33.3, 36.9)
Connections:
- A1 pad 27: +5V -> VCC
- J2 pad 1: +5V -> VCC
- R2 pad 1: +5V -> VCC
- R3 pad 1: +5V -> VCC
- U3 pad 1: Net-(A1-D11) -> Net-(A1-D8)
- U3 pad 13: Net-(J1-Pin_4) -> Net-(J1-Pin_1)
- U3 pad 14: Net-(J1-Pin_3) -> Net-(J1-Pin_2)
- U3 pad 15: Net-(J1-Pin_2) -> Net-(J1-Pin_3)
- U3 pad 16: Net-(J1-Pin_1) -> Net-(J1-Pin_4)
- U3 pad 2: Net-(A1-D10) -> Net-(A1-D9)
- U3 pad 3: Net-(A1-D9) -> Net-(A1-D10)
- U3 pad 4: Net-(A1-D8) -> Net-(A1-D11)
- U4 pad 3: +5V -> VCC
Routing:
- net +5V: track 93.1 -> 0.00 mm, vias 1 -> 0
- net VCC: track 90.3 -> 140.7 mm, vias 0 -> 1
- net Net-(A1-D7): track 55.4 -> 36.9 mm, vias 1 -> 0
- net Net-(A1-D8): track 27.0 -> 20.6 mm
- net Net-(A1-A4): track 72.6 -> 78.6 mm, vias 0 -> 1
- net Net-(A1-D9): track 26.5 -> 20.6 mm
- net Net-(A1-D10): track 26.0 -> 20.8 mm
- net Net-(A1-D11): track 25.5 -> 20.8 mm
- net Net-(J1-Pin_4): track 11.7 -> 8.38 mm
- net Net-(J1-Pin_3): track 10.6 -> 8.36 mm
- net Net-(J1-Pin_1): track 6.93 -> 8.33 mm
- net GND: vias 9 -> 11
Other:
- board text added: "USB"
