File: PCB/KiCad/Splitflap/Splitflap.kicad_sch (KiCad schematic)
At the start: 18 parts, among them J1 Conn_01x05, J2 Conn_01x03, J3_In1 Conn_01x04, J4_Out1 Conn_01x04, Q1 BSS138, Q2 BSS138, U1 ESP8266-01_ESP-01, U2 L7805, U3 ULN2003A, U4 AMS1117-3.3

Commit message: 5v variante
Parts:
- removed C2, C3: C, Capacitor_THT:CP_Radial_D4.0mm_P2.00mm, symbol Device:C
- removed U2: L7805, Package_TO_SOT_THT:TO-220-3_Vertical, symbol Regulator_Linear:L7805
- U3: footprint Package_SO:SOP-16_4.55x10.3mm_P1.27mm -> Package_DIP:DIP-16_W7.62mm
Connections:
- net +5V is gone; now on net VCC: A1.27 (+5V), J2.1 (Pin_1), R2.1, R3.1, U4.3 (VI)
- net at U3.1 (I1): now also A1.11 (D8); no longer A1.14 (D11)
- net at U3.13 (O4): now also J1.1 (Pin_1); no longer J1.4 (Pin_4)
- net at U3.14 (O3): now also J1.2 (Pin_2); no longer J1.3 (Pin_3)
- net at U3.15 (O2): now also J1.3 (Pin_3); no longer J1.2 (Pin_2)
- net at U3.16 (O1): now also J1.4 (Pin_4); no longer J1.1 (Pin_1)
- net at U3.2 (I2): now also A1.12 (D9); no longer A1.13 (D10)
- net at U3.3 (I3): now also A1.13 (D10); no longer A1.12 (D9)
- net at U3.4 (I4): now also A1.14 (D11); no longer A1.11 (D8)
Other:
- moved on the sheet: U3
